File: gurindam.kicad_pcb (KiCad board)
At the start: 2 copper layers, 355.6 x 121.9 mm, 135 parts, among them U1 promicro

Commit message: wired the columns.
Parts:
- moved diode65 269.6 mm to (295.1, 2.24), turned to 90 degrees
- moved diode66 262.3 mm to (299.9, 21.3), turned to 90 degrees
- moved diode6 250.6 mm to (19.1, 7.00), turned to 90 degrees
- moved diode60 236.1 mm to (252.3, 7.00), turned to 90 degrees
- moved diode48 235.6 mm to (217.8, 45.1), turned to 90 degrees
- moved diode37 231.7 mm to (157.9, 17.5), turned to 102 degrees
- moved diode24 230.9 mm to (94.4, 17.2), turned to 78 degrees
- moved diode1 229.8 mm to (0.00, 7.00), turned to 90 degrees
- moved diode57 229.6 mm to (267.8, 45.1), turned to 90 degrees
- moved diode67 229.3 mm to (303.5, 88.0), turned to 90 degrees
- moved diode33 221.9 mm to (139.3, 21.5), turned to 102 degrees
- moved diode55 221.7 mm to (233.2, 7.00), turned to 90 degrees
- moved diode2 220.1 mm to (0.60, 26.1), turned to 90 degrees
- moved diode62 217.9 mm to (304.7, 40.3), turned to 90 degrees
- moved diode10 215.9 mm to (38.5, 5.30), turned to 78 degrees
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Routing:
- net C7: track 0.00 -> 231.2 mm
- net C5: track 0.00 -> 212.5 mm
- net C6: track 0.00 -> 199.6 mm
- net C4: track 0.00 -> 189.9 mm
- net C3: track 0.00 -> 188.8 mm
- net C2: track 0.00 -> 171.3 mm
- net C1: track 0.00 -> 161.3 mm
- net C8: track 0.00 -> 121.1 mm
- net Net-(diode1-Pad1): track 0.00 -> 39.6 mm
- net Net-(diode15-Pad1): track 0.00 -> 39.2 mm
- net Net-(diode41-Pad2): track 0.00 -> 15.3 mm
- net Net-(diode23-Pad2): track 0.00 -> 13.6 mm
- net Net-(diode22-Pad2): track 0.00 -> 11.0 mm
- net Net-(diode20-Pad2): track 0.00 -> 11.0 mm
- net Net-(diode11-Pad2): track 0.00 -> 11.0 mm
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Other:
- board size 355.6 x 121.9 mm -> 335.3 x 116.8 mm

Commit message: finished.
Parts:
- removed the diode28 at (125.7, -42.8)
- removed the switch28 at (109.2, -50.4)
- renumbered diode29 to diode28, diode30 to diode29, diode31 to diode30, diode32 to diode31, diode33 to diode32, diode34 to diode33, diode35 to diode34, diode36 to diode35, diode37 to diode36, diode38 to diode37, diode39 to diode38, diode40 to diode39, diode41 to diode40, diode42 to diode41, diode43 to diode42, diode44 to diode43, diode45 to diode44, diode46 to diode45, diode47 to diode46, diode48 to diode47, diode49 to diode48, diode50 to diode49, diode51 to diode50, diode52 to diode51, diode53 to diode52, diode54 to diode53, diode55 to diode54, diode56 to diode55, diode57 to diode56, diode58 to diode57, diode59 to diode58, diode60 to diode59, diode61 to diode60, diode62 to diode61, diode63 to diode62, diode64 to diode63, diode65 to diode64, diode66 to diode65, diode67 to diode66, switch29 to switch28, switch30 to switch29, switch31 to switch30, switch32 to switch31, switch33 to switch32, switch34 to switch33, switch35 to switch34, switch36 to switch35, switch37 to switch36, switch38 to switch37, switch39 to switch38, switch40 to switch39, switch41 to switch40, switch42 to switch41, switch43 to switch42, switch44 to switch43, switch45 to switch44, switch46 to switch45, switch47 to switch46, switch48 to switch47, switch49 to switch48, switch50 to switch49, switch51 to switch50, switch52 to switch51, switch53 to switch52, switch54 to switch53, switch55 to switch54, switch56 to switch55, switch57 to switch56, switch58 to switch57, switch59 to switch58, switch60 to switch59, switch61 to switch60, switch62 to switch61, switch63 to switch62, switch64 to switch63, switch65 to switch64, switch66 to switch65, switch67 to switch66
Connections:
- U1 pad 10: (no net) -> R3
- U1 pad 11: (no net) -> R2
- U1 pad 12: (no net) -> R1
- U1 pad 13: (no net) -> C8
- U1 pad 14: (no net) -> C7
- U1 pad 15: (no net) -> C6
- U1 pad 16: (no net) -> C5
- U1 pad 17: (no net) -> C4
- U1 pad 18: (no net) -> C1
- U1 pad 19: (no net) -> C2
- U1 pad 2: (no net) -> R9
- U1 pad 20: (no net) -> C3
- U1 pad 5: (no net) -> R8
- U1 pad 6: (no net) -> R7
- U1 pad 7: (no net) -> R6
- U1 pad 8: (no net) -> R5
- U1 pad 9: (no net) -> R4
- diode1 pad 1: Net-(diode1-Pad1) -> R1
- diode10 pad 1: Net-(diode1-Pad1) -> R1
- diode11 pad 1: Net-(diode11-Pad1) -> R3
- diode12 pad 1: Net-(diode12-Pad1) -> R5
- diode13 pad 1: Net-(diode13-Pad1) -> R7
- diode14 pad 1: Net-(diode14-Pad1) -> R9
- diode15 pad 1: Net-(diode15-Pad1) -> R2
- diode16 pad 1: Net-(diode16-Pad1) -> R4
- diode17 pad 1: Net-(diode17-Pad1) -> R6
- diode18 pad 1: Net-(diode18-Pad1) -> R8
- diode19 pad 1: Net-(diode1-Pad1) -> R1
- diode2 pad 1: Net-(diode11-Pad1) -> R3
- diode20 pad 1: Net-(diode11-Pad1) -> R3
- diode21 pad 1: Net-(diode12-Pad1) -> R5
- diode22 pad 1: Net-(diode13-Pad1) -> R7
- diode23 pad 1: Net-(diode14-Pad1) -> R9
- diode24 pad 1: Net-(diode15-Pad1) -> R2
- diode25 pad 1: Net-(diode16-Pad1) -> R4
- diode26 pad 1: Net-(diode17-Pad1) -> R6
- diode27 pad 1: Net-(diode18-Pad1) -> R8
- diode28 pad 1: Net-(diode11-Pad1) -> R3
- diode29 pad 1: Net-(diode12-Pad1) -> R5
- diode3 pad 1: Net-(diode12-Pad1) -> R5
- diode30 pad 1: Net-(diode13-Pad1) -> R7
- diode31 pad 1: Net-(diode14-Pad1) -> R9
- diode32 pad 1: Net-(diode15-Pad1) -> R2
- diode33 pad 1: Net-(diode16-Pad1) -> R4
- diode34 pad 1: Net-(diode17-Pad1) -> R6
- diode35 pad 1: Net-(diode18-Pad1) -> R8
- diode36 pad 1: Net-(diode1-Pad1) -> R1
- diode37 pad 1: Net-(diode11-Pad1) -> R3
- diode38 pad 1: Net-(diode12-Pad1) -> R5
- diode39 pad 1: Net-(diode13-Pad1) -> R7
- diode4 pad 1: Net-(diode13-Pad1) -> R7
- diode40 pad 1: Net-(diode14-Pad1) -> R9
- diode41 pad 1: Net-(diode15-Pad1) -> R2
- diode42 pad 1: Net-(diode16-Pad1) -> R4
- diode43 pad 1: Net-(diode17-Pad1) -> R6
- diode44 pad 1: Net-(diode18-Pad1) -> R8
- diode45 pad 1: Net-(diode1-Pad1) -> R1
- diode46 pad 1: Net-(diode11-Pad1) -> R3
- diode47 pad 1: Net-(diode12-Pad1) -> R5
- diode48 pad 1: Net-(diode13-Pad1) -> R7
- diode49 pad 1: Net-(diode14-Pad1) -> R9
- diode5 pad 1: Net-(diode14-Pad1) -> R9
- diode50 pad 1: Net-(diode15-Pad1) -> R2
- diode51 pad 1: Net-(diode16-Pad1) -> R4
- diode52 pad 1: Net-(diode17-Pad1) -> R6
- diode53 pad 1: Net-(diode18-Pad1) -> R8
- diode54 pad 1: Net-(diode1-Pad1) -> R1
- diode55 pad 1: Net-(diode11-Pad1) -> R3
- diode56 pad 1: Net-(diode12-Pad1) -> R5
- diode57 pad 1: Net-(diode13-Pad1) -> R7
- diode58 pad 1: Net-(diode14-Pad1) -> R9
- diode59 pad 1: Net-(diode15-Pad1) -> R2
- diode6 pad 1: Net-(diode15-Pad1) -> R2
- diode60 pad 1: Net-(diode16-Pad1) -> R4
- diode61 pad 1: Net-(diode17-Pad1) -> R6
- diode62 pad 1: Net-(diode18-Pad1) -> R8
- diode63 pad 1: Net-(diode1-Pad1) -> R1
- diode64 pad 1: Net-(diode11-Pad1) -> R3
- diode65 pad 1: Net-(diode12-Pad1) -> R5
- diode66 pad 1: Net-(diode13-Pad1) -> R7
- diode7 pad 1: Net-(diode16-Pad1) -> R4
- diode8 pad 1: Net-(diode17-Pad1) -> R6
- diode9 pad 1: Net-(diode18-Pad1) -> R8
Routing:
- net R9: track 0.00 -> 405.6 mm, vias 0 -> 1
- net R7: track 0.00 -> 405.3 mm, vias 0 -> 1
- net R5: track 0.00 -> 393.7 mm, vias 0 -> 1
- net R8: track 0.00 -> 363.9 mm, vias 0 -> 1
- net R3: track 0.00 -> 363.7 mm, vias 0 -> 1
- net R6: track 0.00 -> 352.8 mm, vias 0 -> 1
- net R4: track 0.00 -> 295.2 mm, vias 0 -> 1
- net R1: track 0.00 -> 293.9 mm, vias 0 -> 1
- net R2: track 0.00 -> 258.1 mm, vias 0 -> 1
- net C1: track 161.3 -> 360.7 mm
- net C8: track 121.1 -> 313.0 mm
- net C2: track 171.3 -> 330.7 mm
- net C7: track 231.2 -> 387.9 mm
- net C6: track 199.6 -> 339.8 mm
- net C3: track 188.8 -> 291.3 mm
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- added copper zone on B.Cu, net (none)
- added copper zone on F.Cu, net (none)
Other:
- board text added: "apabila banyak berkata-kata di situlah jalan masuk dusta apabila banyak berlebih-lebihan suka itulah tanda hampirkan duka apabila kita kurang siasat itulah tanda pekerjaan hendak sesat apabila anak tidak dilatih jika besar bapanya letih apabila banyak mencacat orang itulah tanda dirinya kurang apabila orang yang banyak tidur sia-sia sahajalah umur apabila mendengar akan khabar menerimanya itu hen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"
- board text added: "apabila terpelihara mata sedikitlah cita-cita apabila terpelihara kuping khabar yang jahat tiadalah damping apabila terpelihara lidah niscaya dapat daripadanya faedah bersungguh-sungguh engkau memeliharakan tangan daripada segala berat dan ringan apabila perut terlalu penuh keluarlah fi�il yang tiada senonoh anggota tengah hendaklah ingat di situlah banyak orang yang hilang semangat hendaklah pel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"
- board text added: "barang siapa khianat akan dirinya apalagi kepada lainnya kepada dirinya ia aniaya orang itu jangan engkau percaya lidah suka membenarkan dirinya daripada yang lain dapat kesalahannya daripada memuji diri hendaklah sabar biar daripada orang datangnya khabar orang yang suka menampakkan jasa setengah daripada syirik mengaku kuasa kejahatan diri sembunyikan kebajikan diri diamkan keaiban orang jangan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"
- board text added: "barang siapa mengenal yang tersebut tahulah ia makna takut barang siapa meninggalkan sembahyang seperti rumah tiada bertiang barang siapa meninggalkan puasa tidaklah mendapat dua termasa barang siapa meninggalkan zakat tiada hartanya beroleh berkat barang siapa meninggalkan haji tiadalah ia menyempurnakan janji"
- board text added: "barang siapa tiada memegang agama sekali-kali tiada boleh dibilangkan nama barang siapa mengenal yang empat maka yaitulah orang yang makrifat barang siapa mengenal Allah suruh dan tegahnya tiada ia menyalah barang siapa mengenal diri maka telah mengenal akan tuhan yang bahri barang siapa mengenal dunia tahulah ia barang yang terperdaya barang siapa mengenal akhirat tahulah ia dunia mudharat"
- board text added: "cahari olehmu akan sahabat yang boleh dijadikan obat cahari olehmu akan guru yang boleh tahukan tiap seteru cahari olehmu akan isteri yang boleh menyerahkan diri cahari olehmu akan kawan pilih segala orang yang setiawan cahari olehmu akan abdi yang ada baik sedikit budi"
- board text added: "hati itu kerajaan di dalam tubuh jikalau zalim segala anggota pun rubuh apabila dengki sudah bertanah datang daripadanya beberapa anak panah mengumpat dan memuji hendaklah pikir di situlah banyak orang yang tergelincir pekerjaan marah jangan dibela nanti hilang akal di kepala jika sedikit pun berbuat bohong boleh diumpamakan mulutnya itu pekung tanda orang yang amat celaka aib dirinya tiada ia sa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"
- board text added: "hendaklah berjasa kepada yang sebangsa hendaklah jadi kepala buang perangai yang cela hendak memegang amanat buanglah khianat hendak marah dahulukan hujjah hendak dimalui jangan memalui hendak ramai murahkan perangai"
- board text added: "jika hendak mengenal orang berbangsa lihat kepada budi dan bahasa jika hendak mengenal orang yang berbahagia sangat memeliharakan yang sia-sia jika hendak mengenal orang mulia lihatlah kepada kelakuan dia jika hendak mengenal orang yang berilmu bertanya dan belajar tiadalah jemu jika hendak mengenal orang yang berakal di dalam dunia mengambil bekal jika hendak mengenal orang yang baik perangai li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"
- board text added: "raja mufakat dengan menteri seperti kebun berpagar duri betul hati kepada raja tanda jadi sebarang kerja hukum adil atas rakyat tanda raja beroleh inayat kasihkan orang yang berilmu tanda rahmat atas dirimu hormat akan orang yang pandai tanda mengenal kasa dan cindai ingatkan dirinya mati itulah asal berbuat bakti akhirat itu terlalu nyata kepada hati yang tidak buta"
- board text added: "tahu pekerjaan tak baik tapi dikerjakan bukannya manusia ia itulah syaitan kejahatan seorang perempaun tua itulah iblis punya penggawa kepada segala hamba-hamba raja di situlah syaitan tempatnya manja kebanyakan orang yang muda-muda di situlah syaitan tempat bergoda perkumpulan laki-laki dengan perempuan di situlah syaitan punya jamuan adapun orang tua yang hemat syaitan tak suka membuat sahabat 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"

Commit message: hotswap socket.
Parts:
- added J1: Conn_01x01, footprints:wirepad, F.Cu at (91.5, -8.15)
- added J2: Conn_01x01, footprints:wirepad, F.Cu at (96.6, -8.15)
- added J3: Conn_01x01, footprints:wirepad, F.Cu at (94.1, -8.15)
- added diode28: diode, footprints:diode, F.Cu at (114.9, 24.8)
- added switch28: switch, footprints:100-socket, F.Cu at (114.5, 14.3)
- added switch68: switch, footprints:reset, F.Cu at (127.7, -7.04)
- switch1, switch10, switch11, switch12, switch13, switch15, switch16, switch17, switch18, switch19, switch20, switch21, switch22, switch24, switch25, switch26, switch27, switch6, switch7, switch8, switch9: footprint footprints:100-minimal -> footprints:100-socket
- switch14, switch2, switch5: footprint footprints:150-minimal -> footprints:150-socket
- switch23: footprint footprints:200-minimal -> footprints:200-socket
- switch29: renamed from switch28; footprint footprints:100-minimal -> footprints:100-socket
- switch3: footprint footprints:175-minimal -> footprints:175-socket
- switch30: renamed from switch29; footprint footprints:100-minimal -> footprints:100-socket
- switch31: renamed from switch30; footprint footprints:100-minimal -> footprints:100-socket
- switch32: renamed from switch31; footprint footprints:100-minimal -> footprints:100-socket
- switch33: renamed from switch32; footprint footprints:100-minimal -> footprints:100-socket
- switch34: renamed from switch33; footprint footprints:100-minimal -> footprints:100-socket
- switch35: renamed from switch34; footprint footprints:100-minimal -> footprints:100-socket
- switch36: renamed from switch35; footprint footprints:100-minimal -> footprints:100-socket
- switch37: renamed from switch36; footprint footprints:100-minimal -> footprints:100-socket
- switch38: renamed from switch37; footprint footprints:100-minimal -> footprints:100-socket
- switch39: renamed from switch38; footprint footprints:100-minimal -> footprints:100-socket
- switch4: footprint footprints:225-minimal -> footprints:225-socket
- switch40: renamed from switch39; footprint footprints:100-minimal -> footprints:100-socket
- switch41: renamed from switch40; footprint footprints:275-minimal -> footprints:275-socket
- switch42: renamed from switch41; footprint footprints:100-minimal -> footprints:100-socket
- switch43: renamed from switch42; footprint footprints:100-minimal -> footprints:100-socket
- switch44: renamed from switch43; footprint footprints:100-minimal -> footprints:100-socket
- switch45: renamed from switch44; footprint footprints:100-minimal -> footprints:100-socket
- switch46: renamed from switch45; footprint footprints:100-minimal -> footprints:100-socket
- switch47: renamed from switch46; footprint footprints:100-minimal -> footprints:100-socket
- switch48: renamed from switch47; footprint footprints:100-minimal -> footprints:100-socket
- switch49: renamed from switch48; footprint footprints:100-minimal -> footprints:100-socket
- switch50: renamed from switch49; footprint footprints:150-minimal -> footprints:150-socket
- switch51: renamed from switch50; footprint footprints:100-minimal -> footprints:100-socket
- switch52: renamed from switch51; footprint footprints:100-minimal -> footprints:100-socket
- switch53: renamed from switch52; footprint footprints:100-minimal -> footprints:100-socket
- switch54: renamed from switch53; footprint footprints:175-minimal -> footprints:175-socket
- switch55: renamed from switch54; footprint footprints:100-minimal -> footprints:100-socket
- switch56: renamed from switch55; footprint footprints:100-minimal -> footprints:100-socket
- switch57: renamed from switch56; footprint footprints:225-minimal -> footprints:225-socket
- switch58: renamed from switch57; footprint footprints:100-minimal -> footprints:100-socket
- switch59: renamed from switch58; footprint footprints:100-minimal -> footprints:100-socket
- switch60: renamed from switch59; footprint footprints:100-minimal -> footprints:100-socket
- switch61: renamed from switch60; footprint footprints:150-minimal -> footprints:150-socket
- switch62: renamed from switch61; footprint footprints:100-minimal -> footprints:100-socket
- switch63: renamed from switch62; footprint footprints:100-minimal -> footprints:100-socket
- switch64: renamed from switch63; footprint footprints:100-minimal -> footprints:100-socket
- switch65: renamed from switch64; footprint footprints:100-minimal -> footprints:100-socket
- switch66: renamed from switch65; footprint footprints:100-minimal -> footprints:100-socket
- switch67: renamed from switch66; footprint footprints:100-minimal -> footprints:100-socket
- moved U1 2.43 mm to (114.4, 5.69)
- renumbered diode28 to diode29, diode29 to diode30, diode30 to diode31, diode31 to diode32, diode32 to diode33, diode33 to diode34, diode34 to diode35, diode35 to diode36, diode36 to diode37, diode37 to diode38, diode38 to diode39, diode39 to diode40, diode40 to diode41, diode41 to diode42, diode42 to diode43, diode43 to diode44, diode44 to diode45, diode45 to diode46, diode46 to diode47, diode47 to diode48, diode48 to diode49, diode49 to diode50, diode50 to diode51, diode51 to diode52, diode52 to diode53, diode53 to diode54, diode54 to diode55, diode55 to diode56, diode56 to diode57, diode57 to diode58, diode58 to diode59, diode59 to diode60, diode60 to diode61, diode61 to diode62, diode62 to diode63, diode63 to diode64, diode64 to diode65, diode65 to diode66, diode66 to diode67
Connections:
- U1 pad 1: (no net) -> embuh
- U1 pad 21: (no net) -> vcc
- U1 pad 22: (no net) -> rst
- U1 pad 23: (no net) -> gnd
- U1 pad 3: (no net) -> gnd
- switch23 pad 1: Net-(diode23-Pad2) -> C3
- switch23 pad 2: C3 -> Net-(diode23-Pad2)
Routing:
- net R8: track 363.9 -> 438.6 mm, vias 1 -> 0
- net C2: track 330.7 -> 262.3 mm
- net R6: track 352.8 -> 416.2 mm, vias 1 -> 0
- net R7: track 405.3 -> 465.5 mm, vias 1 -> 0
- net C1: track 360.7 -> 302.2 mm
- net C3: track 291.3 -> 233.5 mm
- net R4: track 295.2 -> 346.9 mm, vias 1 -> 0
- net R2: track 258.1 -> 299.3 mm, vias 1 -> 0
- net gnd: track 0.00 -> 41.1 mm
- net R3: track 363.7 -> 402.8 mm, vias 1 -> 0
- net C4: track 252.5 -> 290.9 mm
- net R5: track 393.7 -> 428.5 mm, vias 1 -> 0
- net vcc: track 0.00 -> 33.7 mm
- net R9: track 405.6 -> 435.3 mm, vias 1 -> 0
- net C5: track 291.5 -> 310.2 mm
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