File: gurindam.kicad_pcb (KiCad board)
At the start: 2 copper layers, 335.3 x 116.8 mm, 139 parts, among them J1 Conn_01x01, J2 Conn_01x01, J3 Conn_01x01, U1 promicro

Commit message: hm
Routing:
- net Net-(diode41-Pad2): track 15.4 -> 17.0 mm
Changed lines of the file:
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@@
     (thickness 1.6)
     (drawings 18)
-    (tracks 1059)
+    (tracks 1060)
     (zones 0)
     (modules 139)
@@
     (add_net C7)
     (add_net C8)
-    (add_net "Net-(U1-Pad24)")
-    (add_net "Net-(U1-Pad4)")
     (add_net "Net-(diode1-Pad2)")
     (add_net "Net-(diode10-Pad2)")
@@
       (effects (font (size 1.27 1.524) (thickness 0.2032)))
     )
-    (fp_text user 2.75u (at -15.24 8.255 12) (layer Dwgs.User)
-      (effects (font (size 1.524 1.524) (thickness 0.3048)))
-    )
     (fp_line (start -6.985 -4.8768) (end -6.985 -6.985) (layer Eco2.User) (width 0.1524))
     (fp_line (start -8.6106 -4.8768) (end -6.985 -4.8768) (layer Eco2.User) (width 0.1524))
@@
     (fp_line (start 26.19375 -9.525) (end 26.19375 9.525) (layer Dwgs.User) (width 0.1))
     (fp_line (start -26.19375 -9.525) (end 26.19375 -9.525) (layer Dwgs.User) (width 0.1))
+    (fp_text user 2.75u (at -15.24 8.255 12) (layer Dwgs.User)
+      (effects (font (size 1.524 1.524) (thickness 0.3048)))
+    )
     (pad HOLE np_thru_hole circle (at -3.81 -2.54 12) (size 3 3) (drill 3) (layers *.Cu *.Mask))
     (pad HOLE np_thru_hole circle (at 0 0 282) (size 4 4) (drill 4) (layers *.Cu *.Mask))
@@
   (segment (start 179.714555 65.221923) (end 184.720508 70.227876) (width 0.25) (layer B.Cu) (net 40))
   (segment (start 179.714555 61.538795) (end 179.714555 65.221923) (width 0.25) (layer B.Cu) (net 40))
-  (segment (start 165.943574 88.70848) (end 167.950121 88.70848) (width 0.25) (layer B.Cu) (net 41))
-  (segment (start 158.838781 81.603687) (end 165.943574 88.70848) (width 0.25) (layer B.Cu) (net 41))
-  (segment (start 155.490684 81.603687) (end 158.838781 81.603687) (width 0.25) (layer B.Cu) (net 41))
+  (segment (start 167.950121 85.998521) (end 167.950121 88.70848) (width 0.25) (layer B.Cu) (net 41))
+  (segment (start 163.555287 81.603687) (end 167.950121 85.998521) (width 0.25) (layer B.Cu) (net 41))
+  (segment (start 155.490684 81.603687) (end 163.555287 81.603687) (width 0.25) (layer B.Cu) (net 41))
   (segment (start 167.832402 9.320787) (end 172.838355 14.32674) (width 0.25) (layer B.Cu) (net 42))
   (segment (start 167.832402 5.637659) (end 167.832402 9.320787) (width 0.25) (layer B.Cu) (net 42))
@@
   (segment (start 189.9235 54.9656) (end 191.413304 56.455404) (width 0.25) (layer B.Cu) (net 71))
   (segment (start 186.1312 54.9656) (end 189.9235 54.9656) (width 0.25) (layer B.Cu) (net 71))
-  (segment (start 162.2552 92.8116) (end 160.373959 94.692841) (width 0.25) (layer B.Cu) (net 71))
-  (segment (start 169.3672 92.8116) (end 162.2552 92.8116) (width 0.25) (layer B.Cu) (net 71))
-  (segment (start 172.4152 89.7636) (end 169.3672 92.8116) (width 0.25) (layer B.Cu) (net 71))
-  (segment (start 157.152342 94.692841) (end 156.251372 93.791871) (width 0.25) (layer B.Cu) (net 71))
-  (segment (start 160.373959 94.692841) (end 157.152342 94.692841) (width 0.25) (layer B.Cu) (net 71))
-  (segment (start 185.3692 91.9226) (end 177.1142 91.9226) (width 0.25) (layer B.Cu) (net 71))
-  (segment (start 174.9552 89.7636) (end 172.4152 89.7636) (width 0.25) (layer B.Cu) (net 71))
-  (segment (start 177.1142 91.9226) (end 174.9552 89.7636) (width 0.25) (layer B.Cu) (net 71))
-  (segment (start 189.31687 87.97493) (end 185.3692 91.9226) (width 0.25) (layer B.Cu) (net 71))
-  (segment (start 189.31687 59.574178) (end 189.31687 87.97493) (width 0.25) (layer B.Cu) (net 71))
-  (segment (start 191.413304 57.477744) (end 189.31687 59.574178) (width 0.25) (layer B.Cu) (net 71))
-  (segment (start 191.413304 56.455404) (end 191.413304 57.477744) (width 0.25) (layer B.Cu) (net 71))
   (segment (start 192.808724 17.207622) (end 195.1482 19.547098) (width 0.25) (layer B.Cu) (net 71))
   (segment (start 195.1482 19.547098) (end 195.1482 32.1056) (width 0.25) (layer B.Cu) (net 71))
@@
   (segment (start 126.00644 24.543593) (end 119.64119 24.543593) (width 0.25) (layer B.Cu) (net 71))
   (segment (start 117.551199 22.453598) (end 117.551199 16.484601) (width 0.25) (layer B.Cu) (net 71))
+  (segment (start 160.3222 95.0786) (end 157.538101 95.0786) (width 0.25) (layer B.Cu) (net 71))
+  (segment (start 162.5892 92.8116) (end 160.3222 95.0786) (width 0.25) (layer B.Cu) (net 71))
+  (segment (start 172.4152 89.7636) (end 169.3672 92.8116) (width 0.25) (layer B.Cu) (net 71))
+  (segment (start 174.9552 89.7636) (end 172.4152 89.7636) (width 0.25) (layer B.Cu) (net 71))
+  (segment (start 189.31687 87.97493) (end 185.3692 91.9226) (width 0.25) (layer B.Cu) (net 71))
+  (segment (start 189.31687 59.574178) (end 189.31687 87.97493) (width 0.25) (layer B.Cu) (net 71))
+  (segment (start 157.538101 95.0786) (end 156.251372 93.791871) (width 0.25) (layer B.Cu) (net 71))
+  (segment (start 169.3672 92.8116) (end 162.5892 92.8116) (width 0.25) (layer B.Cu) (net 71))
+  (segment (start 177.1142 91.9226) (end 174.9552 89.7636) (width 0.25) (layer B.Cu) (net 71))
+  (segment (start 185.3692 91.9226) (end 177.1142 91.9226) (width 0.25) (layer B.Cu) (net 71))
+  (segment (start 191.413304 57.477744) (end 189.31687 59.574178) (width 0.25) (layer B.Cu) (net 71))
+  (segment (start 191.413304 56.455404) (end 191.413304 57.477744) (width 0.25) (layer B.Cu) (net 71))
   (segment (start 210.253643 12.058113) (end 211.442435 13.246905) (width 0.25) (layer B.Cu) (net 72))
   (segment (start 202.405713 12.058113) (end 210.253643 12.058113) (width 0.25) (layer B.Cu) (net 72))
@@
   (segment (start 95.4532 90.9066) (end 95.4532 92.4306) (width 0.25) (layer F.Cu) (net 81))
   (segment (start 89.828578 85.281978) (end 95.4532 90.9066) (width 0.25) (layer F.Cu) (net 81))
-  (segment (start 114.868383 99.444399) (end 145.081401 99.444399) (width 0.25) (layer F.Cu) (net 81))
-  (segment (start 159.648628 95.123986) (end 161.4932 93.279414) (width 0.25) (layer F.Cu) (net 81))
-  (segment (start 149.401814 95.123986) (end 159.648628 95.123986) (width 0.25) (layer F.Cu) (net 81))
-  (segment (start 145.081401 99.444399) (end 149.401814 95.123986) (width 0.25) (layer F.Cu) (net 81))
-  (segment (start 161.4932 93.279414) (end 161.4932 90.6526) (width 0.25) (layer F.Cu) (net 81))
-  (segment (start 162.991708 80.066939) (end 162.944168 80.019399) (width 0.25) (layer F.Cu) (net 81))
-  (segment (start 162.991708 89.154092) (end 162.991708 80.066939) (width 0.25) (layer F.Cu) (net 81))
-  (segment (start 161.4932 90.6526) (end 162.991708 89.154092) (width 0.25) (layer F.Cu) (net 81))
   (segment (start 169.795147 93.279414) (end 177.374961 85.6996) (width 0.25) (layer F.Cu) (net 81))
   (segment (start 161.4932 93.279414) (end 169.795147 93.279414) (width 0.25) (layer F.Cu) (net 81))
@@
   (segment (start 111.926617 87.693815) (end 114.922023 90.689221) (width 0.25) (layer B.Cu) (net 81))
   (segment (start 111.926617 74.2696) (end 111.926617 87.693815) (width 0.25) (layer B.Cu) (net 81))
+  (segment (start 161.4932 93.6536) (end 161.4932 93.279414) (width 0.25) (layer F.Cu) (net 81))
+  (segment (start 160.022814 95.123986) (end 161.4932 93.6536) (width 0.25) (layer F.Cu) (net 81))
+  (segment (start 149.401814 95.123986) (end 160.022814 95.123986) (width 0.25) (layer F.Cu) (net 81))
+  (segment (start 145.081401 99.444399) (end 149.401814 95.123986) (width 0.25) (layer F.Cu) (net 81))
+  (segment (start 114.868383 99.444399) (end 145.081401 99.444399) (width 0.25) (layer F.Cu) (net 81))
+  (segment (start 161.4932 90.3516) (end 163.1162 88.7286) (width 0.25) (layer F.Cu) (net 81))
+  (segment (start 163.1162 80.191431) (end 162.944168 80.019399) (width 0.25) (layer F.Cu) (net 81))
+  (segment (start 163.1162 88.7286) (end 163.1162 80.191431) (width 0.25) (layer F.Cu) (net 81))
+  (segment (start 161.4932 93.279414) (end 161.4932 90.3516) (width 0.25) (layer F.Cu) (net 81))
   (segment (start 66.454897 49.861036) (end 66.888684 50.294823) (width 0.25) (layer F.Cu) (net 82))
   (segment (start 58.344636 49.861036) (end 66.454897 49.861036) (width 0.25) (layer F.Cu) (net 82))
