File: gurindam.sch (KiCad schematic (older format))
At the start: 135 parts, among them U1 promicro

Commit message: finished.
Parts:
- removed diode28: diode, footprints:diode, symbol rick-kicad-lib:diode
- removed switch28: switch, footprints:100-minimal, symbol rick-kicad-lib:switch
- renumbered diode29 to diode28, diode30 to diode29, diode31 to diode30, diode32 to diode31, diode33 to diode32, diode34 to diode33, diode35 to diode34, diode36 to diode35, diode37 to diode36, diode38 to diode37, diode39 to diode38, diode40 to diode39, diode41 to diode40, diode42 to diode41, diode43 to diode42, diode44 to diode43, diode45 to diode44, diode46 to diode45, diode47 to diode46, diode48 to diode47, diode49 to diode48, diode50 to diode49, diode51 to diode50, diode52 to diode51, diode53 to diode52, diode54 to diode53, diode55 to diode54, diode56 to diode55, diode57 to diode56, diode58 to diode57, diode59 to diode58, diode60 to diode59, diode61 to diode60, diode62 to diode61, diode63 to diode62, diode64 to diode63, diode65 to diode64, diode66 to diode65, diode67 to diode66, switch29 to switch28, switch30 to switch29, switch31 to switch30, switch32 to switch31, switch33 to switch32, switch34 to switch33, switch35 to switch34, switch36 to switch35, switch37 to switch36, switch38 to switch37, switch39 to switch38, switch40 to switch39, switch41 to switch40, switch42 to switch41, switch43 to switch42, switch44 to switch43, switch45 to switch44, switch46 to switch45, switch47 to switch46, switch48 to switch47, switch49 to switch48, switch50 to switch49, switch51 to switch50, switch52 to switch51, switch53 to switch52, switch54 to switch53, switch55 to switch54, switch56 to switch55, switch57 to switch56, switch58 to switch57, switch59 to switch58, switch60 to switch59, switch61 to switch60, switch62 to switch61, switch63 to switch62, switch64 to switch63, switch65 to switch64, switch66 to switch65, switch67 to switch66
Connections:
- net labels added: R1, R2, R3, R4, R5, R6, R7, R8, R9
- wire segments 171 -> 170

Commit message: hotswap socket.
Parts:
- added J1, J2, J3: Conn_01x01, footprints:wirepad, symbol Connector_Generic:Conn_01x01
- added diode28: diode, footprints:diode, symbol rick-kicad-lib:diode
- added switch28: switch, footprints:100-socket, symbol rick-kicad-lib:switch
- added switch68: switch, footprints:reset, symbol rick-kicad-lib:switch
- switch1, switch10, switch11, switch12, switch13, switch15, switch16, switch17, switch18, switch19, switch20, switch21, switch22, switch24, switch25, switch26, switch27, switch6, switch7, switch8, switch9: footprint footprints:100-minimal -> footprints:100-socket
- switch14, switch2, switch5: footprint footprints:150-minimal -> footprints:150-socket
- switch23: footprint footprints:200-minimal -> footprints:200-socket
- switch29: renamed from switch28; footprint footprints:100-minimal -> footprints:100-socket
- switch3: footprint footprints:175-minimal -> footprints:175-socket
- switch30: renamed from switch29; footprint footprints:100-minimal -> footprints:100-socket
- switch31: renamed from switch30; footprint footprints:100-minimal -> footprints:100-socket
- switch32: renamed from switch31; footprint footprints:100-minimal -> footprints:100-socket
- switch33: renamed from switch32; footprint footprints:100-minimal -> footprints:100-socket
- switch34: renamed from switch33; footprint footprints:100-minimal -> footprints:100-socket
- switch35: renamed from switch34; footprint footprints:100-minimal -> footprints:100-socket
- switch36: renamed from switch35; footprint footprints:100-minimal -> footprints:100-socket
- switch37: renamed from switch36; footprint footprints:100-minimal -> footprints:100-socket
- switch38: renamed from switch37; footprint footprints:100-minimal -> footprints:100-socket
- switch39: renamed from switch38; footprint footprints:100-minimal -> footprints:100-socket
- switch4: footprint footprints:225-minimal -> footprints:225-socket
- switch40: renamed from switch39; footprint footprints:100-minimal -> footprints:100-socket
- switch41: renamed from switch40; footprint footprints:275-minimal -> footprints:275-socket
- switch42: renamed from switch41; footprint footprints:100-minimal -> footprints:100-socket
- switch43: renamed from switch42; footprint footprints:100-minimal -> footprints:100-socket
- switch44: renamed from switch43; footprint footprints:100-minimal -> footprints:100-socket
- switch45: renamed from switch44; footprint footprints:100-minimal -> footprints:100-socket
- switch46: renamed from switch45; footprint footprints:100-minimal -> footprints:100-socket
- switch47: renamed from switch46; footprint footprints:100-minimal -> footprints:100-socket
- switch48: renamed from switch47; footprint footprints:100-minimal -> footprints:100-socket
- switch49: renamed from switch48; footprint footprints:100-minimal -> footprints:100-socket
- switch50: renamed from switch49; footprint footprints:150-minimal -> footprints:150-socket
- switch51: renamed from switch50; footprint footprints:100-minimal -> footprints:100-socket
- switch52: renamed from switch51; footprint footprints:100-minimal -> footprints:100-socket
- switch53: renamed from switch52; footprint footprints:100-minimal -> footprints:100-socket
- switch54: renamed from switch53; footprint footprints:175-minimal -> footprints:175-socket
- switch55: renamed from switch54; footprint footprints:100-minimal -> footprints:100-socket
- switch56: renamed from switch55; footprint footprints:100-minimal -> footprints:100-socket
- switch57: renamed from switch56; footprint footprints:225-minimal -> footprints:225-socket
- switch58: renamed from switch57; footprint footprints:100-minimal -> footprints:100-socket
- switch59: renamed from switch58; footprint footprints:100-minimal -> footprints:100-socket
- switch60: renamed from switch59; footprint footprints:100-minimal -> footprints:100-socket
- switch61: renamed from switch60; footprint footprints:150-minimal -> footprints:150-socket
- switch62: renamed from switch61; footprint footprints:100-minimal -> footprints:100-socket
- switch63: renamed from switch62; footprint footprints:100-minimal -> footprints:100-socket
- switch64: renamed from switch63; footprint footprints:100-minimal -> footprints:100-socket
- switch65: renamed from switch64; footprint footprints:100-minimal -> footprints:100-socket
- switch66: renamed from switch65; footprint footprints:100-minimal -> footprints:100-socket
- switch67: renamed from switch66; footprint footprints:100-minimal -> footprints:100-socket
- renumbered diode28 to diode29, diode29 to diode30, diode30 to diode31, diode31 to diode32, diode32 to diode33, diode33 to diode34, diode34 to diode35, diode35 to diode36, diode36 to diode37, diode37 to diode38, diode38 to diode39, diode39 to diode40, diode40 to diode41, diode41 to diode42, diode42 to diode43, diode43 to diode44, diode44 to diode45, diode45 to diode46, diode46 to diode47, diode47 to diode48, diode48 to diode49, diode49 to diode50, diode50 to diode51, diode51 to diode52, diode52 to diode53, diode53 to diode54, diode54 to diode55, diode55 to diode56, diode56 to diode57, diode57 to diode58, diode58 to diode59, diode59 to diode60, diode60 to diode61, diode61 to diode62, diode62 to diode63, diode63 to diode64, diode64 to diode65, diode65 to diode66, diode66 to diode67
Connections:
- net C3: now also switch23.1; no longer switch23.2
- net C4: now also switch28.2
- net R1: now also diode28.1
- net at diode23.2: now also switch23.2; no longer switch23.1
- net embuh: now reaches U1.1 (TX)
- net embuh: now also J3.1 (Pin_1)
- net vcc: now reaches U1.21 (VCC)
- net vcc: now also J2.1 (Pin_1)
- net rst: now reaches U1.22 (RST)
- net rst: now also switch68.2
- net gnd: now reaches U1.23 (GND)
- net gnd: now also U1.3 (GND), J1.1 (Pin_1), switch68.1
- new net: diode28.2, switch28.1
Other:
- moved on the sheet: U1, switch23
